Commit message: fix: update

File: velodyne_description/urdf/VLP-32.urdf.xacro (robot description, xacro)
@@ -26,10 +26,10 @@
       <visual>
         <geometry>
-          <mesh filename="package://velodyne_description/meshes/VLP32_base_1.dae"/>
+          <mesh filename="package://velodyne_description/meshes/VLP16_base_1.dae"/>
         </geometry>
       </visual>
       <visual>
         <geometry>
-          <mesh filename="package://velodyne_description/meshes/VLP32_base_2.dae"/>
+          <mesh filename="package://velodyne_description/meshes/VLP16_base_2.dae"/>
         </geometry>
       </visual>
